File: Platine/federkontaktplatine_oben/federkontaktplatine_oben.kicad_sch (KiCad schematic)
At the start: 17 parts, among them J2 Conn_01x08

Commit message: Platinen update
Parts:
- removed J2: Conn_01x08, Connector_Molex:Molex_Micro-Fit_3.0_43650-0810_1x08-1MP_P3.00mm_Horizontal, symbol Connector_Generic:Conn_01x08
- added H1 (x4), H2 (x3), H3 (x4): MountingHole, MountingHole:MountingHole_3.2mm_M3_DIN965, symbol Mechanical:MountingHole
- added J1: Conn_01x10, Connector_Molex:MOLEX_436501012, symbol Connector_Generic:Conn_01x10
- added J2: Conn_01x07, Connector_Molex:MOLEX_436500712, symbol Connector_Generic:Conn_01x07
- added J3, J4: Conn_02x10_Odd_Even, Connector_PinSocket_2.54mm:PinSocket_2x10_P2.54mm_Vertical_SMD, symbol Connector_Generic:Conn_02x10_Odd_Even
Connections:
- net at TP11.1, TP12.1: now also J4.3 (Pin_3)
- net at TP13.1, TP14.1: now also J4.1 (Pin_1)
- net at TP15.1, TP16.1: now also J4.9 (Pin_9)
- net at TP1.1, TP2.1: now also J4.15 (Pin_15)
- net at TP5.1, TP6.1: now also J4.11 (Pin_11)
- net at TP3.1, TP4.1: now also J4.13 (Pin_13)
- net at TP10.1, TP9.1: now also J4.5 (Pin_5)
- net at TP7.1, TP8.1: now also J4.7 (Pin_7)
- new net: J1.1 (Pin_1), J3.2 (Pin_2)
- new net: J1.10 (Pin_10), J3.20 (Pin_20)
- new net: J1.2 (Pin_2), J3.4 (Pin_4)
- new net: J1.3 (Pin_3), J3.6 (Pin_6)
- new net: J1.4 (Pin_4), J3.8 (Pin_8)
- new net: J1.5 (Pin_5), J3.10 (Pin_10)
- new net: J1.6 (Pin_6), J3.12 (Pin_12)
- new net: J1.7 (Pin_7), J3.14 (Pin_14)
- new net: J1.8 (Pin_8), J3.16 (Pin_16)
- new net: J1.9 (Pin_9), J3.18 (Pin_18)
- new net: J2.1 (Pin_1), J4.2 (Pin_2)
- new net: J2.2 (Pin_2), J4.4 (Pin_4)
- new net: J2.3 (Pin_3), J4.6 (Pin_6)
- new net: J2.4 (Pin_4), J4.8 (Pin_8)
- new net: J2.5 (Pin_5), J4.10 (Pin_10)
- new net: J2.6 (Pin_6), J4.12 (Pin_12)
- new net: J2.7 (Pin_7), J4.14 (Pin_14)
- new net GND: J3.1 (Pin_1), J3.11 (Pin_11), J3.13 (Pin_13), J3.15 (Pin_15), J3.17 (Pin_17), J3.19 (Pin_19), J3.3 (Pin_3), J3.5 (Pin_5), J3.7 (Pin_7), J3.9 (Pin_9)

Commit message: platinen
Parts:
- added H2: MountingHole, MountingHole:MountingHole_3.2mm_M3_DIN965, symbol Mechanical:MountingHole
Changed lines of the file:
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@@
+    )
+  )
+  (symbol (lib_id "Mechanical:MountingHole") (at 54.61 60.96 0) (unit 1)
+    (in_bom yes) (on_board yes) (dnp no) (fields_autoplaced)
+    (property "Reference" "H2" (at 57.15 59.6899 0)
+      (effects (font (size 1.27 1.27)) (justify left))
+    )
+    (property "Value" "MountingHole" (at 57.15 62.2299 0)
+      (effects (font (size 1.27 1.27)) (justify left))
+    )
+    (property "Footprint" "MountingHole:MountingHole_3.2mm_M3_DIN965" (at 54.61 60.96 0)
+      (effects (font (size 1.27 1.27)) hide)
+    )
+    (property "Datasheet" "~" (at 54.61 60.96 0)
+      (effects (font (size 1.27 1.27)) hide)
+    )
+    (instances
+      (project "FTCMS_V2.2"
+        (path "/30da9297-09e7-47e7-9d66-9d536b8d0426"
+          (reference "H2") (unit 1)
+        )
+      )
+      (project "federkontaktplatine_oben"
+        (path "/67804148-9fb2-45a4-a226-f3c6005bfe46"
+          (reference "H11") (unit 1)
+        )
+      )
+      (project "FTCMS_PCB_v2.2"
+        (path "/83a6a285-13b6-4ec8-ae72-c2fe713cc487"
+          (reference "H2") (unit 1)
+        )
+      )
     )
   )
