File: Platine/federkontaktplatine_oben/federkontaktplatine_oben.kicad_pcb (KiCad board)
At the start: 2 copper layers, 256 x 137.5 mm, 32 parts, among them J1 Conn_01x10, J2 Conn_01x07, J3 Conn_02x10_Odd_Even, J4 Conn_02x10_Odd_Even

Commit message: Kabelstrang
Parts:
- moved H12 20.2 mm to (255.5, 98.8)
- moved H4 20.2 mm to (40.5, 58.8)
- moved H5 20.2 mm to (40.5, 138.8)
- moved H6 20.2 mm to (40.5, 98.8)
- moved H8 20.2 mm to (255.5, 58.8)
- moved H9 20.2 mm to (255.5, 138.8)
Changed lines of the file:
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@@
   (net 31 "Net-(J1-Pin_1)")
   (footprint "MountingHole:MountingHole_3.2mm_M3_DIN965" (layer "F.Cu")
-    (at 252.5 38.75)
+    (at 255.5 58.75)
     (descr "Mounting Hole 3.2mm, no annular, M3, DIN965")
     (tags "mounting hole 3.2mm no annular m3 din965")
@@
   )
   (footprint "MountingHole:MountingHole_3.2mm_M3_DIN965" (layer "F.Cu")
-    (at 252.5 78.75)
+    (at 255.5 98.75)
     (descr "Mounting Hole 3.2mm, no annular, M3, DIN965")
     (tags "mounting hole 3.2mm no annular m3 din965")
@@
   )
   (footprint "MountingHole:MountingHole_3.2mm_M3_DIN965" (layer "F.Cu")
-    (at 43.5 78.75)
+    (at 40.5 98.75)
     (descr "Mounting Hole 3.2mm, no annular, M3, DIN965")
     (tags "mounting hole 3.2mm no annular m3 din965")
@@
   )
   (footprint "MountingHole:MountingHole_3.2mm_M3_DIN965" (layer "F.Cu")
-    (at 252.5 118.75)
+    (at 255.5 138.75)
     (descr "Mounting Hole 3.2mm, no annular, M3, DIN965")
     (tags "mounting hole 3.2mm no annular m3 din965")
@@
   )
   (footprint "MountingHole:MountingHole_3.2mm_M3_DIN965" (layer "F.Cu")
-    (at 43.5 38.75)
+    (at 40.5 58.75)
     (descr "Mounting Hole 3.2mm, no annular, M3, DIN965")
     (tags "mounting hole 3.2mm no annular m3 din965")
@@
   )
   (footprint "MountingHole:MountingHole_3.2mm_M3_DIN965" (layer "F.Cu")
-    (at 43.5 118.75)
-    (descr "Mounting Hole 3.2mm, no annular, M3, DIN965")
-    (tags "mounting hole 3.2mm no annular m3 din965")
+    (at 40.5 138.75)
+    (descr "Mounting Hole 3.2mm, no annular, M3, DIN965")
+    (tags "mounting hole 3.2mm no annular m3 din965")
